File: CAD/KiCad/keyboard.kicad_pcb (KiCad board)
At the start: 2 copper layers, 307.2 x 148.8 mm, 202 parts, among them J1 OLED_128x32, J2 Conn_01x02_Socket, J3 4P4C, J4 OLED_128x32, J5 Conn_01x02_Socket, J6 4P4C, SW1 Switch, SW2 SW_SPDT, SW3 Switch, SW4 SW_SPDT, U1 XIAO-HALF-HOLE-23P, U3 XIAO-HALF-HOLE-23P

Commit message: update pcb
Parts:
- removed REF** (x4): mousebites 2mm, PCM_marbastlib-various:mousebites_2mm
Other:
- board size 307.2 x 148.8 mm -> 305 x 125.4 mm
- board text removed: "JLCJLCJLCJLC"
